File: Template_Puzzles/Wire_Puzzle/Wire_Puzzle.sch (EAGLE design)
At the start: 24 parts, among them Q1 2N7002

Commit message: Wire_Puzzle progress
Parts:
- removed J0, J1, J2, J3, J4, J5, J6, J7: (no value), SparkFun-Connectors:CONN_04
- added D1: 1N4001, Diodes:1N4004
- added IC1: 7805T, linear:7805T
- added R3: 330R, Resistor:R_AXIAL-7.2MM-PITCH
- added U$10, U$11, U$12, U$13, U$14, U$15, U$16, U$17: 1X02, Adam's Parts (work):1X02
- added U$18, U$19, U$20, U$21, U$22, U$23, U$24, U$25, U$26, U$27: 1X03, Adam's Parts (work):1X03
- FRAME1: value FRAME-LETTER -> FRAME-LEDGER; device Adam's Parts (work):FRAME-LETTER -> Adam's Parts (work):FRAME-LEDGER
- Q1: value 2N7002 -> 2N7000
Connections:
- new net N$5: LED1.A, R3.2
- net 5V: now also D1.C, IC1.VO, R3.1, U$18.2, U$19.2, U$20.2, U$21.2, U$22.2, U$23.2, U$24.2, U$25.2, U$26.2, U$27.2
- net A: now also U$10.2; no longer J0.2
- net A0: now also U$27.3
- net B: now also U$11.2; no longer J1.2
- net C: now also U$12.2; no longer J2.2
- net D: now also U$13.2; no longer J3.2
- net D0: now also U$18.3, U$7.2
- net D1: now also U$19.3
- net D2: now also U$20.3, U$3.SER; no longer U$7.2
- net D3: now also U$21.3
- net D4: now also U$22.3
- net D5: now also U$23.3
- net D6: now also U$24.3
- net D7: now also U$25.3; no longer U$3.SER
- net D8: now also U$26.3
- net E: now also U$14.2; no longer J4.2
- net F: now also U$15.2; no longer J5.2
- net G: now also U$16.2; no longer J6.2
- net GND: now also IC1.GND, LED1.C, U$18.1, U$19.1, U$20.1, U$21.1, U$22.1, U$23.1, U$24.1, U$25.1, U$26.1, U$27.1; no longer J0.3, J0.4, J1.3, J1.4, J2.3, J2.4, J3.3, J3.4, J4.3, J4.4, J5.3, J5.4, J6.3, J6.4, J7.3, J7.4
- net H: now also U$17.2; no longer J7.2
- net N$4: now also D1.A
- net QA: now also U$10.1; no longer J0.1
- net QB: now also U$11.1; no longer J1.1
- net QC: now also U$12.1; no longer J2.1
- net QD: now also U$13.1; no longer J3.1
- net QE: now also U$14.1; no longer J4.1
- net QF: now also U$15.1; no longer J5.1
- net QG: now also U$16.1; no longer J6.1
- net QH: now also U$17.1; no longer J7.1
- net VCC: now also IC1.VI
Other:
- note added: "CAP 0.1uF"
- note added: "CAP 0.33uF"
- note added: "Diode for reverse polarity protection MOSFET for IO pin separation"
- note added: "Input Power Regulation"
- note added: "NodeMCU IO Breakout Pins"
- note added: "Pin arragement matches Neopixel LED strip"
- note added: "Power Switch"
- note added: "Puzzle Wire Jumpers"
- note added: "Speaker can not exceed 3W power unless amplifying the signal externally"
- note removed: "Power"
- note removed: "Shift Register IO Pins"
- moved on the sheet: LED1, LED2, Q1, R1, R2, RN1, U$1, U$2, U$3, U$6, U$7, U$8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

Commit message: Progress, added audio amp, power
Parts:
- added C1: 1000uF, adafruit:CPOL-USE5-10.5
- added C2: 100uF, adafruit:CPOL-USE5-10.5
- added C3: 0.1uF, capacitor-wima:C2.5/2
- added C4: 0.33uF, rcl:CPOL-USE2-5
- added C5: 0.1uF, rcl:CPOL-USE2-5
- added D2: 1N4001, Diodes:1N4004
- added R4, R5: 1K, Resistor:R_AXIAL-7.2MM-PITCH
- added R6: 10R, Resistor:R_AXIAL-7.2MM-PITCH
- added S1: (no value), Adam's Parts (work):SWITCH_SLIDING_SSP1S1
- added U1: LM386N, SparkFun-IC-Amplifiers:LM386
- added VR1: 10k, SparkFun-Resistors:TRIMPOT-PTH-10MM-KNOB-1/2W-10%
- R2: value (none) -> 330R
Connections:
- new net AUDIO: R4.1, R5.1, VR1.WIPER
- new net N$10: C3.2, R6.1
- new net N$11: R5.2, U$5.P$13
- new net N$12: U1.+IN, VR1.CW
- new net N$13: S1.P, U$2.2
- new net N$14: C2.+, U1.BP
- new net N$9: C1.-, U$9.1
- net 5V: now also C5.+, D2.A
- net GND: now also C2.-, C4.-, C5.-, R6.2, U$9.2, U1.-IN, U1.V-
- net N$7: now also C1.+, C3.1, U1.OUT; no longer U$5.P$16, U$9.1
- net N$8: now also R4.2, U$5.P$12; no longer U$5.P$14, U$9.2
- net VCC: now also C4.+, D2.C, S1.S, U1.V+; no longer U$2.2
Other:
- note added: "Audio Amplifier"
- note added: "C1 smooths the audio and can vary, but must be greater than 250uF. C2 filters amplified VCC noise. C3 filters high frequency audio noise. Potentiometer CW turn increases volume."
- note added: "Diode protects circuit from negative polarity. LED indicates power output to board. C4 and C5 must be as physically close to regulator as possible."
- note added: "Drive pin D1 HIGH to activate. MOSFET for IO pin separation. LED indicates relay state. Diode protects circuit from negative discharge on relay close."
- note added: "Music Player"
- note added: "Regulated Output"
- note added: "Shift register pins can remain disconnected when unused. All shift register clocks are tied together to minimize the control pins required. Shift registers are always active, and all resets and inhibitors are disabled."
- note removed: "All shift register clocks are tied together to minimize the control pins required."
- note removed: "CAP 0.1uF"
- note removed: "CAP 0.33uF"
- note removed: "DFMini Player"
- note removed: "Diode for reverse polarity protection MOSFET for IO pin separation"
- note removed: "Power Switch"
- note removed: "Shift register pins can remain disconnected when unused."
- note removed: "Shift registers are always active, and all resets and inhibitors are disabled."
- note removed: "Speaker can not exceed 3W power unless amplifying the signal externally"
- moved on the sheet: U$2, U$9

Commit message: Finished wire puzzle
Parts:
- R2, R3: value 330R -> 330
- R6: value 10R -> 10
Connections:
- net GND: now also U$4.G_2, U$4.G_4, U$9.1; no longer U$9.2
- net N$9: now also U$9.2; no longer U$9.1
Other:
- note added: "Escape Room "Connect the Wires" Puzzle Board"
- note added: "Place barrel jacks in a grid, connect the solution pairs to a pair of letters in the included PUZZLE WIRES section of the board. Play some music and sound effects on the DFMini Player. Trigger an electromagnet or other device with the relay. Flash some lights with Neopixel LEDs."
- moved on the sheet: C1, C2, C3, C4, C5, D1, D2, LED1, LED2, Q1, R1, R2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

Commit message: Cleaned up Wire_Puzzle PCB labels, added DC power jack
Parts:
- removed U$2: TERMINAL_BLOCK_2P, Adam's Parts (work):TERMINAL_BLOCK_2P
- added J1: POWER_JACK_PJ-037A, Adam's Parts (work):POWER_JACK_PJ-037A
Connections:
- net 5V: now also U$4.VU
- net GND: now also J1.2; no longer U$2.1
- net N$13: now also J1.1; no longer U$2.2
Other:
- note added: "C1 smooths the audio and can vary, but must be greater than 250uF. C2 filters amplified VCC noise. C3 filters high frequency audio noise. Speaker impedance must exceed 4R. Potentiometer CW turn increases volume."
- note added: "Diode protects 5V circuit from inverted VCC. LED indicates power output to board. C4 and C5 must be as physically close to regulator as possible."
- note removed: "C1 smooths the audio and can vary, but must be greater than 250uF. C2 filters amplified VCC noise. C3 filters high frequency audio noise. Potentiometer CW turn increases volume."
- note removed: "Diode protects circuit from negative polarity. LED indicates power output to board. C4 and C5 must be as physically close to regulator as possible."
- moved on the sheet: R4, R5
